Commit message: Second

File: description/sja_gazebo.xacro (robot description, xacro)
@@ -14,15 +14,15 @@
             (which robot_state_publisher can then use to broadcast the approprate tf). -->
     <gazebo>
-        <plugin name="gazebo_ros_joint_state_publisher"
-            filename="libgazebo_ros_joint_state_publisher.so">
-            <update_rate>20</update_rate>
-            <joint_name>joint1</joint_name>
-            <joint_name>joint2</joint_name>
-        </plugin>
-    </gazebo>
-    <gazebo>
-        <plugin name="gazebo_ros_joint_pose_trajectory"
-            filename="libgazebo_ros_joint_pose_trajectory.so">
-            <update_rate>20</update_rate>
+        <plugin name="gazebo_ros2_control" filename="libgazebo_ros2_control.so">
+            <robot_namespace>/</robot_namespace>
+            <update_rate>100</update_rate>
+            <joint>
+                <name>joint1</name>
+                <hardwareInterface>PositionJointInterface</hardwareInterface>
+            </joint>
+            <joint>
+                <name>joint2</name>
+                <hardwareInterface>PositionJointInterface</hardwareInterface>
+            </joint>
         </plugin>
     </gazebo>
